File: hardware/pcb/ecocell-carrier.kicad_pcb (KiCad board)
At the start: 2 copper layers, 100 x 80 mm, 20 parts, among them J1 PIR, J10 EMIT-40k, J2 HYDRO, J3 ULTRA, J4 I2C-BME280, J5 I2C-BH1750, J6 I2C-AD7746, J7 UART, J8 SPI, J9 5V-IN, Q1 2N7000, U1A XIAO-L, U1B XIAO-R

Commit message: EcoCell carrier v2: field-protection layer + production fab package
Upgrade the generated carrier toward a deployable node: rugged Phoenix
screw-terminal 5V input feeding polyfuse, SMAJ5.0A rail TVS and SS14
reverse-polarity Schottky; PESD5V0 ESD clamps on the three exposed head
signal lines; 3V3 power LED; three fiducials for the PCBA line. Board
regenerates from tools/pcb/gen_carrier.py; kicad-cli DRC reports 0
violations and 0 unconnected items. Gerbers, drill, 25-line BOM and
12-part CPL re-exported; renders refreshed.

Adds hardware/FIELD-KIT.md — the complete sourcing matrix splitting
Seeed-assembled parts from plug-in/field items (XIAO, heads, radio,
power, enclosure) plus the first-article test plan. Docs updated to
state clearly: fab-ready, not yet production-proven until a fabricated
unit passes bench + E0 field validation and compliance review.

Generated with [Devin](https://devin.ai)

Co-Authored-By: Devin <158243242+devin-ai-integration[bot]@users.noreply.github.com>
Parts:
- added D2: SS14, D_SMA, F.Cu at (59.0, 74.5)
- added D3: SMAJ5.0A, D_SMA, F.Cu at (68.0, 76.0)
- added D4: PESD5V0, D_SOD-323, F.Cu at (15.5, 22.5)
- added D5: PESD5V0, D_SOD-323, F.Cu at (15.5, 32.5)
- added D6: PESD5V0, D_SOD-323, F.Cu at (15.5, 42.5)
- added F1: 0.75A, Fuse_1206_3216Metric, F.Cu at (74.0, 74.5)
- added FID1: FID, Fiducial_1mm_Mask3mm, F.Cu at (10.0, 10.0)
- added FID2: FID, Fiducial_1mm_Mask3mm, F.Cu at (90.0, 10.0)
- added FID3: FID, Fiducial_1mm_Mask3mm, F.Cu at (10.0, 66.0)
- added J11: 5V-SCREW, TerminalBlock_Phoenix_MKDS-1,5-2_1x02_P5.00mm_Horizontal, F.Cu at (80.0, 74.5)
- added LED1: PWR-GRN, LED_0805_2012Metric, F.Cu at (76.0, 20.0)
- added R2: 1k, R_0805_2012Metric, F.Cu at (71.5, 20.0)
Routing:
- net GND: track 367.3 -> 423.0 mm, vias 8 -> 11
- net VPROT: track 0.00 -> 13.1 mm
- net D2_ULTRA: track 33.5 -> 40.5 mm
- net D1_HYDRO: track 30.9 -> 37.9 mm
- net D0_PIR: track 30.0 -> 37.0 mm
- net +3V3: track 310.2 -> 315.2 mm
- net VIN: track 0.00 -> 4.60 mm
- net +5V: track 173.7 -> 176.7 mm, vias 0 -> 1
- net LEDPWR: track 0.00 -> 2.62 mm
Other:
- board text added: "5V-IN protected"
- board text added: "PWR"

Commit message: Make the field node genuinely orderable: MPNs, click-path, provisioning
- Fix Q1 value 2N7000 -> 2N7002 (SOT-23 footprint; 2N7000 is TO-92)
- FIELD-KIT.md: concrete manufacturer part numbers for every PCBA line,
  real XIAO/part numbers for plug-ins, named power-module options
- New PROVISIONING.md: flash -> identity -> consent defaults -> edge
  pairing -> field commissioning, the software half of buy-and-deploy
- PCB.md: explicit Seeed Fusion ordering click-path
- Gerbers/drill/render re-exported; DRC still 0/0

Generated with [Devin](https://devin.ai)

Co-Authored-By: Devin <158243242+devin-ai-integration[bot]@users.noreply.github.com>
Parts:
- Q1: value 2N7000 -> 2N7002
